Commit message: edit: add MoveIt configuration files for JAKA-Lumi-sensors-v3

File: src/robot_description/JAKA-Lumi-sensors-v3/urdf/jaka_lumi_sensors_v3.urdf (robot description, URDF)
Before this commit: robot JAKA-Lumi-sensors-v3, 26 links, 25 joints
Links:
- added link world
Joints:
- added joint world_to_base_joint: type fixed, parent world, child base_link, origin xyz=0 0 0 rpy=0 0 0
