Commit message: adjust: tidy up the directory structure of robot_description

File: src/robot_description/urdf/jaka_lumi_sensors_v3.urdf (robot description, URDF)
Before this commit: robot JAKA-Lumi-sensors-v3, 27 links, 26 joints
Links:
- link Camera1_Link: geometry collision mesh filename=package://robot_description/meshes/Camera1_Link.STL; visual mesh filename=package://robot_description/meshes/Camera1_Link.STL
- link Camera2_Link: geometry collision mesh filename=package://robot_description/meshes/Camera2_Link.STL; visual mesh filename=package://robot_description/meshes/Camera2_Link.STL
- link Camera3_Link: geometry collision mesh filename=package://robot_description/meshes/Camera3_Link.STL; visual mesh filename=package://robot_description/meshes/Camera3_Link.STL
- link Radar_Link: geometry collision mesh filename=package://robot_description/meshes/Radar_Link.STL; visual mesh filename=package://robot_description/meshes/Radar_Link.STL
- link base_link: geometry collision mesh filename=package://robot_description/meshes/base_link.STL; visual mesh filename=package://robot_description/meshes/base_link.STL
- link link_1: geometry collision mesh filename=package://robot_description/meshes/link_1.STL; visual mesh filename=package://robot_description/meshes/link_1.STL
- link link_2: geometry collision mesh filename=package://robot_description/meshes/link_2.STL; visual mesh filename=package://robot_description/meshes/link_2.STL
- link link_3: geometry collision mesh filename=package://robot_description/meshes/link_3.STL; visual mesh filename=package://robot_description/meshes/link_3.STL
- link link_4: geometry collision mesh filename=package://robot_description/meshes/link_4.STL; visual mesh filename=package://robot_description/meshes/link_4.STL
- link link_a1: geometry collision mesh filename=package://robot_description/meshes/link_a1.STL; visual mesh filename=package://robot_description/meshes/link_a1.STL
- link link_a2: geometry collision mesh filename=package://robot_description/meshes/link_a2.STL; visual mesh filename=package://robot_description/meshes/link_a2.STL
- link link_a3: geometry collision mesh filename=package://robot_description/meshes/link_a3.STL; visual mesh filename=package://robot_description/meshes/link_a3.STL
- link link_a4: geometry collision mesh filename=package://robot_description/meshes/link_a4.STL; visual mesh filename=package://robot_description/meshes/link_a4.STL
- link link_a5: geometry collision mesh filename=package://robot_description/meshes/link_a5.STL; visual mesh filename=package://robot_description/meshes/link_a5.STL
- link link_a6: geometry collision mesh filename=package://robot_description/meshes/link_a6.STL; visual mesh filename=package://robot_description/meshes/link_a6.STL
- link link_at: geometry collision mesh filename=package://robot_description/meshes/link_at.STL; visual mesh filename=package://robot_description/meshes/link_at.STL
- link pw1_Link1: geometry collision mesh filename=package://robot_description/meshes/pw1_Link1.STL; visual mesh filename=package://robot_description/meshes/pw1_Link1.STL
- link pw1_Link2: geometry collision mesh filename=package://robot_description/meshes/pw1_Link2.STL; visual mesh filename=package://robot_description/meshes/pw1_Link2.STL
- link pw2_Link1: geometry collision mesh filename=package://robot_description/meshes/pw2_Link1.STL; visual mesh filename=package://robot_description/meshes/pw2_Link1.STL
- link pw2_Link2: geometry collision mesh filename=package://robot_description/meshes/pw2_Link2.STL; visual mesh filename=package://robot_description/meshes/pw2_Link2.STL
- link pw3_Link1: geometry collision mesh filename=package://robot_description/meshes/pw3_Link1.STL; visual mesh filename=package://robot_description/meshes/pw3_Link1.STL
- link pw3_Link2: geometry collision mesh filename=package://robot_description/meshes/pw3_Link2.STL; visual mesh filename=package://robot_description/meshes/pw3_Link2.STL
- link pw4_Link1: geometry collision mesh filename=package://robot_description/meshes/pw4_Link1.STL; visual mesh filename=package://robot_description/meshes/pw4_Link1.STL
- link pw4_Link2: geometry collision mesh filename=package://robot_description/meshes/pw4_Link2.STL; visual mesh filename=package://robot_description/meshes/pw4_Link2.STL
- link wheel_l: geometry collision mesh filename=package://robot_description/meshes/wheel_l.STL; visual mesh filename=package://robot_description/meshes/wheel_l.STL
- link wheel_r: geometry collision mesh filename=package://robot_description/meshes/wheel_r.STL; visual mesh filename=package://robot_description/meshes/wheel_r.STL

Commit message: fix: fix l_a4 pitch angle problem and remove convertor function in arm_controller

File: src/robot_description/urdf/jaka_lumi_sensors_v3.urdf (robot description, URDF)
Before this commit: robot JAKA-Lumi-sensors-v3, 27 links, 26 joints
Joints:
- joint l_a4: origin xyz=0.1303 0 0.0185 rpy=-1.5708 0 -1.5708 -> xyz=0.1303 0 0.0185 rpy=-1.5708 3.1416 -1.5708
